Commit message: 🧪 test(RL): DQN-2015
testing DQN using pytorch

File: Tests/urdf_generator/hebi/test.urdf (robot description, URDF)
Before this commit: robot UNNAMED_0, 7 links, 6 joints
Links:
- added link Arm/J4_wrist/INPUT_INTERFACE, mass 0.315; collision mesh filename=meshes/X5.stl scale=0.001 0.001 0.001; visual mesh filename=meshes/X5.stl scale=0.001 0.001 0.001
- added link end_effector/INPUT_INTERFACE, mass 0.0; visual box size=0.001 0.001 0.001
Joints:
- added joint Arm/J4_wrist: type continuous, parent Arm/J4_wrist/INPUT_INTERFACE, child end_effector/INPUT_INTERFACE, origin xyz=0 0 0.031 rpy=0 0 0, axis 0 0 1, limit effort=2.5 velocity=9.425
- added joint elbow_wrist/OUTPUT_JOINT: type fixed, parent elbow_wrist/INPUT_INTERFACE, child Arm/J4_wrist/INPUT_INTERFACE, origin xyz=0.325 -0.0 0.04 rpy=0 0 0
